File: pendulum_controller/HKCV4.brd (EAGLE design)
At the start: 57 x 37 mm, 56 parts, among them Q1 TPH, Q2 TPH, Q3 TPH, Q4 TPH, Q5 TPH, Q6 TPH, U1 LTC2851MPDDPBF

Commit message: fixing controller BOM mistake
Parts:
- C1, C11, C12, C13, C14, C15, C16, C18, C8: value 10 -> 10 uF
- C10: value 1uF -> 1 uF
- C17: value .1 uF -> 10 uF
- C2, C4: device rcl:C0603K -> rcl:C0402K
- C27, C31, C32, VREFCAP: value 100nF -> .1 uF
- C41: value 100nF -> .1 uF; device rcl:C0402 -> rcl:C0402K
- C9: value 4.7 -> 4.7 uF
- MC1: value 1uf -> 1 uF; device rcl:C0402 -> rcl:C0402K
- moved C41 2.70 mm to (16.9, 9.11)
- moved C12 2.70 mm to (9.59, -8.55)
- moved C13 2.70 mm to (7.49, -8.55)
- moved C14 2.70 mm to (3.47, -8.40)
- moved C27 2.70 mm to (12.2, 13.5)
- moved C3 2.70 mm to (-15.4, 9.54)
- moved C4 2.70 mm to (-11.3, 4.93)
- moved C9 2.70 mm to (6.48, 13.5)
- moved L1 2.70 mm to (-14.9, 6.35)
- moved Q1 2.70 mm to (-13.9, -13.1)
- moved Q2 2.70 mm to (-8.50, -14.6)
- moved Q4 2.70 mm to (-2.80, -14.6)
- moved Q6 2.70 mm to (14.0, -12.7)
- moved R22 2.70 mm to (9.41, 14.8)
- moved C1 2.70 mm to (1.53, -8.40)
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